File: hardware/rev-a/lora-node.kicad_sch (KiCad schematic)
At the start: 0 parts

Commit message: Schematic: cosmetic pass over the sheet artwork
Other:
- note added: "5 RF"
- note removed: "2 Power"
- note removed: "3 MCU"
- note removed: "4 Radio"
- note removed: "5 Sensors"
- note removed: "6 RF"
Changed lines of the file:
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@@
 		(comment 1 "Off-grid agricultural sensor node - 868 MHz LoRa + BLE")
 	)
-	(text "5  Sensors"
+	(text "4  Sensors"
 		(exclude_from_sim no)
 		(at 25 198 0)
@@
 		)
 	)
-	(text "4  Radio"
+	(text "3  Radio"
 		(exclude_from_sim no)
 		(at 25 193 0)
@@
 		)
 	)
-	(text "3  MCU"
+	(text "2  MCU"
 		(exclude_from_sim no)
 		(at 25 188 0)
@@
 		)
 	)
-	(text "2  Power"
+	(text "1  Power"
 		(exclude_from_sim no)
 		(at 25 183 0)
@@
 		)
 	)
-	(text "6  RF"
+	(text "5  RF"
 		(exclude_from_sim no)
 		(at 25 203 0)
@@
 		)
 	)
-	(text "6  RF"
+	(text "5  RF"
 		(exclude_from_sim no)
 		(at 25 114 0)
@@
 			(project "lora-node"
 				(path "/1f7b3c40-5a2e-5d18-9c6b-3e9a4d2f7b60"
-					(page "4")
+					(page "3")
 				)
 			)
@@
 			(project "lora-node"
 				(path "/1f7b3c40-5a2e-5d18-9c6b-3e9a4d2f7b60"
-					(page "5")
+					(page "4")
 				)
 			)
@@
 			(project "lora-node"
 				(path "/1f7b3c40-5a2e-5d18-9c6b-3e9a4d2f7b60"
-					(page "2")
+					(page "1")
 				)
 			)
@@
 			(project "lora-node"
 				(path "/1f7b3c40-5a2e-5d18-9c6b-3e9a4d2f7b60"
-					(page "3")
+					(page "2")
 				)
 			)
@@
 			(project "lora-node"
 				(path "/1f7b3c40-5a2e-5d18-9c6b-3e9a4d2f7b60"
-					(page "6")
+					(page "5")
 				)
 			)
@@
 	(sheet_instances
 		(path "/"
-			(page "1")
-		)
-	)
+			(page "0")
+		)
+	)
